File: kicad proj/driver_4q_2k20/bridge_gate_driver.sch (KiCad schematic (older format))
At the start: 0 parts

Commit message: adicionado arquivos step, docs e footprints
Changed lines of the file:
@@
 $EndSheet
 $Sheet
-S 4050 650  1400 500
+S 4100 700  1400 500
 U 5EDC1083
 F0 "PWM Modulator" 50
 F1 "pwm_modulator.sch" 50
-F2 "PWM_SIG" O L 4050 1050 50
+F2 "PWM_SIG" O L 4100 950 50
 $EndSheet
-Wire Wire Line
-	4050 1050 3050 1050
-Wire Wire Line
-	3050 1050 3050 1300
-Wire Wire Line
-	3050 1300 2350 1300
 $Sheet
-S 4050 1450 950  400
+S 4100 1450 950  400
 U 5EDD5CBB
 F0 "Motor Direction Control" 50
 F1 "motor_dir.sch" 50
-F2 "DIR" O L 4050 1600 50
+F2 "DIR" O L 4100 1650 50
 $EndSheet
-Wire Wire Line
-	2350 1400 3850 1400
-Wire Wire Line
-	3850 1400 3850 1600
-Wire Wire Line
-	3850 1600 4050 1600
 $Sheet
-S 1050 2250 1150 350
+S 1150 2300 1150 350
 U 5EDE0D36
 F0 "Power Supply" 50
 F1 "power_supply.sch" 50
 $EndSheet
+Wire Wire Line
+	2350 1300 3050 1300
+Wire Wire Line
+	3050 1300 3050 950
+Wire Wire Line
+	3050 950  4100 950
+Wire Wire Line
+	2350 1400 3050 1400
+Wire Wire Line
+	3050 1400 3050 1650
+Wire Wire Line
+	3050 1650 4100 1650
 $EndSCHEMATC
